File: video9958/design/kicad/v9958video/v9958video.kicad_pcb (KiCad board)
At the start: 2 copper layers, 97 x 89 mm, 53 parts, among them IC1 V9958, IC2 ATF16V8BQL-15, IC3 ATF16V8BQL-15, J1 Conn_02x32_Odd_Even, J2 Conn_02x06_Counter_Clockwise, J3 DIN-6, Q1 21.477MHz, Q2 2N3904, Q3 2N3906, Q4 2N3906, Q5 2N3906, U1 41464, U2 41464, U3 41464, U4 41464, U5 41464, U6 41464

Commit message: First round fixes
Parts:
- removed the C19 at (118.7, 73.0)
- added C14: 100uF, Capacitor_THT:CP_Radial_D5.0mm_P2.50mm, F.Cu at (122.7, 73.0)
- added C21: 10uF, Capacitor_THT:CP_Radial_D5.0mm_P2.50mm, F.Cu at (116.0, 73.0)
- C15: renamed from C13; footprint rosco_m68k:C-Electolytic-2,5-5 -> Capacitor_THT:CP_Radial_D6.3mm_P2.50mm
- C16: renamed from C14; footprint rosco_m68k:C-Electolytic-2,5-5 -> Capacitor_THT:CP_Radial_D6.3mm_P2.50mm
- C17: renamed from C16; footprint rosco_m68k:C-Electolytic-2,5-5 -> Capacitor_THT:CP_Radial_D6.3mm_P2.50mm
- C18: footprint rosco_m68k:C-Electolytic-2,5-5 -> Capacitor_THT:CP_Radial_D6.3mm_P2.50mm
- C19: renamed from C15; footprint rosco_m68k:C-Electolytic-2,5-5 -> Capacitor_THT:CP_Radial_D5.0mm_P2.50mm
- C20: renamed from C17; footprint rosco_m68k:C-Electolytic-2,5-5 -> Capacitor_THT:CP_Radial_D5.0mm_P2.50mm
- moved C18 3.65 mm to (115.0, 56.8)
- moved C15 2.82 mm to (122.0, 56.8)
- moved C17 1.97 mm to (129.0, 56.8)
- moved C20 1.64 mm to (129.3, 73.0)
- moved C16 1.03 mm to (136.0, 56.8)
- moved C19 1.03 mm to (136.0, 73.0)
- renumbered C5 to C1, C4 to C10, C1 to C11, C2 to C12, C20 to C13, C6 to C2, C7 to C4, C8 to C5, C9 to C6, C10 to C7, C11 to C8, C12 to C9, IC2 to IC1, IC3 to IC2, IC1 to IC3, R13 to R11, R14 to R12, R7 to R13, R11 to R14, R8 to R5, R12 to R6, R5 to R7, R6 to R8
Routing:
- net VCC: track 475.2 -> 593.2 mm
- net GND: track 572.7 -> 680.4 mm, vias 0 -> 1
- net OBLUE: track 13.7 -> 19.7 mm
- net OCSYNC: track 11.3 -> 16.9 mm, vias 0 -> 1
- net Net-(C18-Pad1): track 37.0 -> 42.2 mm
- net Net-(C17-Pad1): track 26.2 -> 30.0 mm
- net Net-(Q2-Pad2): track 49.3 -> 52.6 mm, vias 0 -> 1
- net OGREEN: track 14.3 -> 16.0 mm
- net Net-(C15-Pad1): track 41.8 -> 42.8 mm
- net /v9958-output/GREEN: track 78.5 -> 79.4 mm
- net Net-(C21-Pad2): track 32.8 -> 32.2 mm
- net /v9958-output/RED: track 82.2 -> 82.7 mm
- removed copper zone on B.Cu, net GND
- removed copper zone on F.Cu, net GND
Other:
- board size 97 x 89 mm -> 102 x 89 mm
- board text added: "Revision 1 (June 2020)"
- board text removed: "Revision 0 (prototype)"

Commit message: Rev 1 - Four layer board
Parts:
- added C14: 100uF, Capacitor_THT:CP_Radial_D5.0mm_P2.50mm, F.Cu at (113.4, 103.2)
- added C15: 100uF, Capacitor_THT:CP_Radial_D5.0mm_P2.50mm, F.Cu at (113.4, 111.0)
- added C24: 100nF, Capacitor_THT:C_Rect_L7.0mm_W2.5mm_P5.00mm, F.Cu at (113.9, 67.3)
- added C25: 100nF, Capacitor_THT:C_Rect_L7.0mm_W2.5mm_P5.00mm, F.Cu at (114.6, 96.9)
- added REF**: WEEE-Logo_4.2x6mm_SilkScreen, Symbol:WEEE-Logo_4.2x6mm_SilkScreen, B.Cu at (212.0, 35.0)
- renumbered C9 to C10, C13 to C11, C11 to C12, C12 to C13, C15 to C16, C16 to C17, C17 to C18, C18 to C19, C19 to C20, C20 to C21, C21 to C22, C14 to C23, C4 to C3, C5 to C4, C6 to C5, C7 to C6, C3 to C7, C10 to C8, C8 to C9
Routing:
- net GND: track 680.4 -> 0.33 mm, vias 1 -> 0
- net VCC: track 593.2 -> 12.0 mm
- net Net-(C19-Pad1): track 42.2 -> 40.8 mm
- net Net-(Q2-Pad2): track 52.6 -> 53.2 mm
- added copper zone on In1.Cu, net GND
- added copper zone on In2.Cu, net VCC
Other:
- board size 102 x 89 mm -> 106 x 89 mm
- copper layers 2 -> 4
