File: video9958/design/kicad/v9958video/output.sch (KiCad schematic (older format))
At the start: 27 parts, among them J2 Conn_02x06_Counter_Clockwise, J3 DIN-6, Q2 2N3904, Q3 2N3906, Q4 2N3906, Q5 2N3906

Commit message: First cut PCB
Parts:
- C13, C14, C15, C16, C17, C18, C19: footprint (none) -> rosco_m68k:C-Electolytic-2,5-5
- J2: footprint (none) -> Connector_PinHeader_2.54mm:PinHeader_2x06_P2.54mm_Vertical
- J3: footprint (none) -> rosco_m68k:din-6
- R10, R11, R12, R13, R14, R15, R2, R4, R5, R6, R7, R8, R9: footprint (none) -> rosco_m68k:R-0207_10
- R3: value R -> 100R; footprint (none) -> rosco_m68k:R-0207_10
Connections:
- net BLUE: now also J2.2 (Pin_2); no longer J2.6 (Pin_6)
- net EXT_VIDEO: now also J2.5 (Pin_5); no longer J2.11 (Pin_11)
- net EXT_VSYNC: now also J2.9 (Pin_9); no longer J2.10 (Pin_10)
- net GND: now also J2.11 (Pin_11); no longer J2.7 (Pin_7)
- net GREEN: now also J2.6 (Pin_6); no longer J2.5 (Pin_5)
- net HSYNC: now also J2.10 (Pin_10); no longer J2.9 (Pin_9)
- net NTSCCLK: now also J2.7 (Pin_7); no longer J2.2 (Pin_2)
Changed lines of the file:
@@
 F 0 "C13" V 3205 6450 50  0000 C CNN
 F 1 "220uF" V 3114 6450 50  0000 C CNN
-F 2 "" H 2988 6300 50  0001 C CNN
+F 2 "rosco_m68k:C-Electolytic-2,5-5" H 2988 6300 50  0001 C CNN
 F 3 "~" H 2950 6450 50  0001 C CNN
 	1    2950 6450
@@
 P 2450 6800
 F 0 "R3" H 2520 6846 50  0000 L CNN
-F 1 "R" H 2520 6755 50  0000 L CNN
-F 2 "" V 2380 6800 50  0001 C CNN
+F 1 "100R" H 2520 6755 50  0000 L CNN
+F 2 "rosco_m68k:R-0207_10" V 2380 6800 50  0001 C CNN
 F 3 "~" H 2450 6800 50  0001 C CNN
 	1    2450 6800
@@
 F 0 "R2" V 1493 6050 50  0000 C CNN
 F 1 "1K" V 1584 6050 50  0000 C CNN
-F 2 "" V 1630 6050 50  0001 C CNN
+F 2 "rosco_m68k:R-0207_10" V 1630 6050 50  0001 C CNN
 F 3 "~" H 1700 6050 50  0001 C CNN
 	1    1700 6050
@@
 F 0 "J3" H 5350 4381 50  0000 C CNN
 F 1 "DIN-6" H 5350 4290 50  0000 C CNN
-F 2 "" H 5350 3900 50  0001 C CNN
-F 3 "http://www.mouser.com/ds/2/18/40_c091_abd_e-75918.pdf" H 5350 3900 50  0001 C CNN
+F 2 "rosco_m68k:din-6" H 5350 3900 50  0001 C CNN
+F 3 "https://docs.rs-online.com/e199/0900766b8153d253.pdf" H 5350 3900 50  0001 C CNN
 	1    5350 3900
 	1    0    0    -1
@@
 F 0 "C18" V 8095 4550 50  0000 C CNN
 F 1 "220uF" V 8186 4550 50  0000 C CNN
-F 2 "" H 8388 4400 50  0001 C CNN
+F 2 "rosco_m68k:C-Electolytic-2,5-5" H 8388 4400 50  0001 C CNN
 F 3 "~" H 8350 4550 50  0001 C CNN
 	1    8350 4550
@@
 F 0 "R13" H 9470 4346 50  0000 L CNN
 F 1 "27K" H 9470 4255 50  0000 L CNN
-F 2 "" V 9330 4300 50  0001 C CNN
+F 2 "rosco_m68k:R-0207_10" V 9330 4300 50  0001 C CNN
 F 3 "~" H 9400 4300 50  0001 C CNN
 	1    9400 4300
@@
 F 0 "R12" H 8920 4346 50  0000 L CNN
 F 1 "100R" H 8920 4255 50  0000 L CNN
-F 2 "" V 8780 4300 50  0001 C CNN
+F 2 "rosco_m68k:R-0207_10" V 8780 4300 50  0001 C CNN
 F 3 "~" H 8850 4300 50  0001 C CNN
 	1    8850 4300
@@
 F 0 "R14" H 9470 5096 50  0000 L CNN
 F 1 "12K" H 9470 5005 50  0000 L CNN
-F 2 "" V 9330 5050 50  0001 C CNN
+F 2 "rosco_m68k:R-0207_10" V 9330 5050 50  0001 C CNN
 F 3 "~" H 9400 5050 50  0001 C CNN
 	1    9400 5050
@@
 F 0 "C19" V 9495 4800 50  0000 C CNN
 F 1 "10uF" V 9586 4800 50  0000 C CNN
-F 2 "" H 9788 4650 50  0001 C CNN
+F 2 "rosco_m68k:C-Electolytic-2,5-5" H 9788 4650 50  0001 C CNN
 F 3 "~" H 9750 4800 50  0001 C CNN
 	1    9750 4800
@@
 F 0 "R15" H 10220 5096 50  0000 L CNN
 F 1 "1K" H 10220 5005 50  0000 L CNN
-F 2 "" V 10080 5050 50  0001 C CNN
+F 2 "rosco_m68k:R-0207_10" V 10080 5050 50  0001 C CNN
 F 3 "~" H 10150 5050 50  0001 C CNN
 	1    10150 5050
@@
 F 0 "C16" V 8095 2900 50  0000 C CNN
 F 1 "220uF" V 8186 2900 50  0000 C CNN
-F 2 "" H 8388 2750 50  0001 C CNN
+F 2 "rosco_m68k:C-Electolytic-2,5-5" H 8388 2750 50  0001 C CNN
 F 3 "~" H 8350 2900 50  0001 C CNN
 	1    8350 2900
@@
 F 0 "R9" H 9470 2696 50  0000 L CNN
 F 1 "27K" H 9470 2605 50  0000 L CNN
-F 2 "" V 9330 2650 50  0001 C CNN
+F 2 "rosco_m68k:R-0207_10" V 9330 2650 50  0001 C CNN
 F 3 "~" H 9400 2650 50  0001 C CNN
 	1    9400 2650
@@
 F 0 "R8" H 8920 2696 50  0000 L CNN
 F 1 "100R" H 8920 2605 50  0000 L CNN
-F 2 "" V 8780 2650 50  0001 C CNN
+F 2 "rosco_m68k:R-0207_10" V 8780 2650 50  0001 C CNN
 F 3 "~" H 8850 2650 50  0001 C CNN
 	1    8850 2650
@@
 F 0 "R10" H 9470 3446 50  0000 L CNN
 F 1 "12K" H 9470 3355 50  0000 L CNN
-F 2 "" V 9330 3400 50  0001 C CNN
+F 2 "rosco_m68k:R-0207_10" V 9330 3400 50  0001 C CNN
 F 3 "~" H 9400 3400 50  0001 C CNN
 	1    9400 3400
@@
 F 0 "C17" V 9495 3150 50  0000 C CNN
 F 1 "10uF" V 9586 3150 50  0000 C CNN
-F 2 "" H 9788 3000 50  0001 C CNN
+F 2 "rosco_m68k:C-Electolytic-2,5-5" H 9788 3000 50  0001 C CNN
 F 3 "~" H 9750 3150 50  0001 C CNN
 	1    9750 3150
@@
 F 0 "R11" H 10220 3446 50  0000 L CNN
 F 1 "1K" H 10220 3355 50  0000 L CNN
-F 2 "" V 10080 3400 50  0001 C CNN
+F 2 "rosco_m68k:R-0207_10" V 10080 3400 50  0001 C CNN
 F 3 "~" H 10150 3400 50  0001 C CNN
 	1    10150 3400
@@
 F 0 "C14" V 8095 1300 50  0000 C CNN
 F 1 "220uF" V 8186 1300 50  0000 C CNN
-F 2 "" H 8388 1150 50  0001 C CNN
+F 2 "rosco_m68k:C-Electolytic-2,5-5" H 8388 1150 50  0001 C CNN
 F 3 "~" H 8350 1300 50  0001 C CNN
 	1    8350 1300
@@
 F 0 "R5" H 9470 1096 50  0000 L CNN
 F 1 "27K" H 9470 1005 50  0000 L CNN
-F 2 "" V 9330 1050 50  0001 C CNN
+F 2 "rosco_m68k:R-0207_10" V 9330 1050 50  0001 C CNN
 F 3 "~" H 9400 1050 50  0001 C CNN
 	1    9400 1050
@@
 F 0 "R4" H 8920 1096 50  0000 L CNN
 F 1 "100R" H 8920 1005 50  0000 L CNN
-F 2 "" V 8780 1050 50  0001 C CNN
+F 2 "rosco_m68k:R-0207_10" V 8780 1050 50  0001 C CNN
 F 3 "~" H 8850 1050 50  0001 C CNN
 	1    8850 1050
@@
 F 0 "R6" H 9470 1846 50  0000 L CNN
 F 1 "12K" H 9470 1755 50  0000 L CNN
-F 2 "" V 9330 1800 50  0001 C CNN
+F 2 "rosco_m68k:R-0207_10" V 9330 1800 50  0001 C CNN
 F 3 "~" H 9400 1800 50  0001 C CNN
 	1    9400 1800
@@
 F 0 "C15" V 9495 1550 50  0000 C CNN
 F 1 "10uF" V 9586 1550 50  0000 C CNN
-F 2 "" H 9788 1400 50  0001 C CNN
+F 2 "rosco_m68k:C-Electolytic-2,5-5" H 9788 1400 50  0001 C CNN
 F 3 "~" H 9750 1550 50  0001 C CNN
 	1    9750 1550
@@
 F 0 "R7" H 10220 1846 50  0000 L CNN
 F 1 "1K" H 10220 1755 50  0000 L CNN
-F 2 "" V 10080 1800 50  0001 C CNN
+F 2 "rosco_m68k:R-0207_10" V 10080 1800 50  0001 C CNN
 F 3 "~" H 10150 1800 50  0001 C CNN
 	1    10150 1800
@@
 $EndComp
 Text HLabel 3400 2000 2    50   Input ~ 0
-HSYNC
+EXT_VSYNC
 Text HLabel 1450 1900 0    50   UnSpc ~ 0
 GND
@@
 CSYNC
 Text HLabel 1450 2200 0    50   Input ~ 0
-BLUE
+GREEN
 Text HLabel 1450 2100 0    50   Input ~ 0
-GREEN
+EXT_VIDEO
 Text HLabel 1450 2000 0    50   Input ~ 0
 RED
@@
 RGB Extension Header
 Text HLabel 1450 1800 0    50   Input ~ 0
+BLUE
+Text HLabel 3400 1900 2    50   Output ~ 0
+HSYNC
+Text HLabel 3400 1800 2    50   Input ~ 0
+GND
+Text HLabel 3400 2200 2    50   UnSpc ~ 0
 NTSCCLK
-Text HLabel 3400 1900 2    50   Output ~ 0
-EXT_VSYNC
-Text HLabel 3400 1800 2    50   Input ~ 0
-EXT_VIDEO
-Text HLabel 3400 2200 2    50   UnSpc ~ 0
-GND
 Text HLabel 3400 1700 2    50   UnSpc ~ 0
 VCC
@@
 F 0 "J2" H 2450 2317 50  0000 C CNN
 F 1 "Conn_02x06_Counter_Clockwise" H 2450 2226 50  0000 C CNN
-F 2 "" H 2400 1900 50  0001 C CNN
+F 2 "Connector_PinHeader_2.54mm:PinHeader_2x06_P2.54mm_Vertical" H 2400 1900 50  0001 C CNN
 F 3 "~" H 2400 1900 50  0001 C CNN
 	1    2400 1900

Commit message: First round fixes
Parts:
- added C14: 100uF, Capacitor_THT:CP_Radial_D5.0mm_P2.50mm, symbol Device:CP
- C15: renamed from C13; footprint rosco_m68k:C-Electolytic-2,5-5 -> Capacitor_THT:CP_Radial_D6.3mm_P2.50mm
- C16: renamed from C14; footprint rosco_m68k:C-Electolytic-2,5-5 -> Capacitor_THT:CP_Radial_D6.3mm_P2.50mm
- C17: renamed from C16; footprint rosco_m68k:C-Electolytic-2,5-5 -> Capacitor_THT:CP_Radial_D6.3mm_P2.50mm
- C18: footprint rosco_m68k:C-Electolytic-2,5-5 -> Capacitor_THT:CP_Radial_D6.3mm_P2.50mm
- C19: renamed from C15; footprint rosco_m68k:C-Electolytic-2,5-5 -> Capacitor_THT:CP_Radial_D5.0mm_P2.50mm
- C20: renamed from C17; footprint rosco_m68k:C-Electolytic-2,5-5 -> Capacitor_THT:CP_Radial_D5.0mm_P2.50mm
- C21: renamed from C19; footprint rosco_m68k:C-Electolytic-2,5-5 -> Capacitor_THT:CP_Radial_D5.0mm_P2.50mm
- renumbered R13 to R11, R14 to R12, R7 to R13, R11 to R14, R8 to R5, R12 to R6, R5 to R7, R6 to R8
Connections:
- net GND: now also C14.2
- net VCC: now also C14.1
Changed lines of the file:
@@
 	2800 6450 2450 6450
 $Comp
-L Device:CP C13
+L Device:CP C15
 U 1 1 5EB8D33A
 P 2950 6450
-F 0 "C13" V 3205 6450 50  0000 C CNN
+F 0 "C15" V 3205 6450 50  0000 C CNN
 F 1 "220uF" V 3114 6450 50  0000 C CNN
-F 2 "rosco_m68k:C-Electolytic-2,5-5" H 2988 6300 50  0001 C CNN
+F 2 "Capacitor_THT:CP_Radial_D6.3mm_P2.50mm" H 2988 6300 50  0001 C CNN
 F 3 "~" H 2950 6450 50  0001 C CNN
 	1    2950 6450
@@
 Wire Wire Line
 	8850 4450 8850 4550
-$Comp
-L Device:CP C18
-U 1 1 5EB704E7
-P 8350 4550
-F 0 "C18" V 8095 4550 50  0000 C CNN
-F 1 "220uF" V 8186 4550 50  0000 C CNN
-F 2 "rosco_m68k:C-Electolytic-2,5-5" H 8388 4400 50  0001 C CNN
-F 3 "~" H 8350 4550 50  0001 C CNN
-	1    8350 4550
-	0    1    1    0
-$EndComp
 Wire Wire Line
 	9400 4450 9400 4800
@@
 	10550 4050 9400 4050
 $Comp
-L Device:R R13
+L Device:R R11
 U 1 1 5EB704DB
 P 9400 4300
-F 0 "R13" H 9470 4346 50  0000 L CNN
+F 0 "R11" H 9470 4346 50  0000 L CNN
 F 1 "27K" H 9470 4255 50  0000 L CNN
 F 2 "rosco_m68k:R-0207_10" V 9330 4300 50  0001 C CNN
@@
 $EndComp
 $Comp
-L Device:R R12
+L Device:R R6
 U 1 1 5EB704D5
 P 8850 4300
-F 0 "R12" H 8920 4346 50  0000 L CNN
+F 0 "R6" H 8920 4346 50  0000 L CNN
 F 1 "100R" H 8920 4255 50  0000 L CNN
 F 2 "rosco_m68k:R-0207_10" V 8780 4300 50  0001 C CNN
@@
 $EndComp
 $Comp
-L Device:R R14
+L Device:R R12
 U 1 1 5EB704B6
 P 9400 5050
-F 0 "R14" H 9470 5096 50  0000 L CNN
+F 0 "R12" H 9470 5096 50  0000 L CNN
 F 1 "12K" H 9470 5005 50  0000 L CNN
 F 2 "rosco_m68k:R-0207_10" V 9330 5050 50  0001 C CNN
@@
 $EndComp
 $Comp
-L Device:CP C19
+L Device:CP C21
 U 1 1 5EB704B0
 P 9750 4800
-F 0 "C19" V 9495 4800 50  0000 C CNN
+F 0 "C21" V 9495 4800 50  0000 C CNN
 F 1 "10uF" V 9586 4800 50  0000 C CNN
-F 2 "rosco_m68k:C-Electolytic-2,5-5" H 9788 4650 50  0001 C CNN
+F 2 "Capacitor_THT:CP_Radial_D5.0mm_P2.50mm" H 9788 4650 50  0001 C CNN
 F 3 "~" H 9750 4800 50  0001 C CNN
 	1    9750 4800
@@
 	8850 2800 8850 2900
 $Comp
-L Device:CP C16
+L Device:CP C17
 U 1 1 5EB5A4E3
 P 8350 2900
-F 0 "C16" V 8095 2900 50  0000 C CNN
+F 0 "C17" V 8095 2900 50  0000 C CNN
 F 1 "220uF" V 8186 2900 50  0000 C CNN
-F 2 "rosco_m68k:C-Electolytic-2,5-5" H 8388 2750 50  0001 C CNN
+F 2 "Capacitor_THT:CP_Radial_D6.3mm_P2.50mm" H 8388 2750 50  0001 C CNN
 F 3 "~" H 8350 2900 50  0001 C CNN
 	1    8350 2900
@@
 $EndComp
 $Comp
-L Device:R R8
+L Device:R R5
 U 1 1 5EB5A4D1
 P 8850 2650
-F 0 "R8" H 8920 2696 50  0000 L CNN
+F 0 "R5" H 8920 2696 50  0000 L CNN
 F 1 "100R" H 8920 2605 50  0000 L CNN
 F 2 "rosco_m68k:R-0207_10" V 8780 2650 50  0001 C CNN
@@
 $EndComp
 $Comp
-L Device:CP C17
+L Device:CP C20
 U 1 1 5EB5A4AC
 P 9750 3150
-F 0 "C17" V 9495 3150 50  0000 C CNN
+F 0 "C20" V 9495 3150 50  0000 C CNN
 F 1 "10uF" V 9586 3150 50  0000 C CNN
-F 2 "rosco_m68k:C-Electolytic-2,5-5" H 9788 3000 50  0001 C CNN
+F 2 "Capacitor_THT:CP_Radial_D5.0mm_P2.50mm" H 9788 3000 50  0001 C CNN
 F 3 "~" H 9750 3150 50  0001 C CNN
 	1    9750 3150
@@
 $EndComp
 $Comp
-L Device:R R11
+L Device:R R14
 U 1 1 5EB5A4A6
 P 10150 3400
-F 0 "R11" H 10220 3446 50  0000 L CNN
+F 0 "R14" H 10220 3446 50  0000 L CNN
 F 1 "1K" H 10220 3355 50  0000 L CNN
 F 2 "rosco_m68k:R-0207_10" V 10080 3400 50  0001 C CNN
@@
 	8850 1200 8850 1300
 $Comp
-L Device:CP C14
+L Device:CP C16
 U 1 1 5EB51CD3
 P 8350 1300
-F 0 "C14" V 8095 1300 50  0000 C CNN
+F 0 "C16" V 8095 1300 50  0000 C CNN
 F 1 "220uF" V 8186 1300 50  0000 C CNN
-F 2 "rosco_m68k:C-Electolytic-2,5-5" H 8388 1150 50  0001 C CNN
+F 2 "Capacitor_THT:CP_Radial_D6.3mm_P2.50mm" H 8388 1150 50  0001 C CNN
 F 3 "~" H 8350 1300 50  0001 C CNN
 	1    8350 1300
@@
 	10550 800  9400 800
 $Comp
-L Device:R R5
+L Device:R R7
 U 1 1 5EB4F451
 P 9400 1050
-F 0 "R5" H 9470 1096 50  0000 L CNN
+F 0 "R7" H 9470 1096 50  0000 L CNN
 F 1 "27K" H 9470 1005 50  0000 L CNN
 F 2 "rosco_m68k:R-0207_10" V 9330 1050 50  0001 C CNN
@@
 $EndComp
 $Comp
-L Device:R R6
+L Device:R R8
 U 1 1 5EB48A0B
 P 9400 1800
-F 0 "R6" H 9470 1846 50  0000 L CNN
+F 0 "R8" H 9470 1846 50  0000 L CNN
 F 1 "12K" H 9470 1755 50  0000 L CNN
 F 2 "rosco_m68k:R-0207_10" V 9330 1800 50  0001 C CNN
@@
 $EndComp
 $Comp
-L Device:CP C15
+L Device:CP C19
 U 1 1 5EB4735D
 P 9750 1550
-F 0 "C15" V 9495 1550 50  0000 C CNN
+F 0 "C19" V 9495 1550 50  0000 C CNN
 F 1 "10uF" V 9586 1550 50  0000 C CNN
-F 2 "rosco_m68k:C-Electolytic-2,5-5" H 9788 1400 50  0001 C CNN
+F 2 "Capacitor_THT:CP_Radial_D5.0mm_P2.50mm" H 9788 1400 50  0001 C CNN
 F 3 "~" H 9750 1550 50  0001 C CNN
 	1    9750 1550
@@
 $EndComp
 $Comp
-L Device:R R7
+L Device:R R13
 U 1 1 5EB46462
 P 10150 1800
-F 0 "R7" H 10220 1846 50  0000 L CNN
+F 0 "R13" H 10220 1846 50  0000 L CNN
 F 1 "1K" H 10220 1755 50  0000 L CNN
 F 2 "rosco_m68k:R-0207_10" V 10080 1800 50  0001 C CNN
@@
 Wire Wire Line
 	2700 1700 3400 1700
+$Comp
+L Device:CP C14
+U 1 1 5ECAC019
+P 2200 3800
+F 0 "C14" H 2318 3846 50  0000 L CNN
+F 1 "100uF" H 2318 3755 50  0000 L CNN
+F 2 "Capacitor_THT:CP_Radial_D5.0mm_P2.50mm" H 2238 3650 50  0001 C CNN
+F 3 "~" H 2200 3800 50  0001 C CNN
+	1    2200 3800
+	1    0    0    -1
+$EndComp
+Wire Wire Line
+	2200 3350 2200 3650
+Wire Wire Line
+	2200 3950 2200 4250
+Text HLabel 2200 3350 1    50   UnSpc ~ 0
+VCC
+Text HLabel 2200 4250 3    50   UnSpc ~ 0
+GND
+$Comp
+L Device:CP C18
+U 1 1 5EB704E7
+P 8350 4550
+F 0 "C18" V 8095 4550 50  0000 C CNN
+F 1 "220uF" V 8186 4550 50  0000 C CNN
+F 2 "Capacitor_THT:CP_Radial_D6.3mm_P2.50mm" H 8388 4400 50  0001 C CNN
+F 3 "~" H 8350 4550 50  0001 C CNN
+	1    8350 4550
+	0    1    1    0
+$EndComp
 $EndSCHEMATC
