File: video9958/design/kicad/v9958video/v9958video.sch (KiCad schematic (older format))
At the start: 29 parts, among them IC1 ATF16V8BQL-15, IC2 ATF16V8BQL-15, IC3 V9958, J1 Conn_02x32_Odd_Even, Q1 21.477MHz, U1 41464, U2 41464, U3 41464, U4 41464, U5 41464, U6 41464

Commit message: Final tweaks
Parts:
- renumbered IC3 to IC1, IC1 to IC2, IC2 to IC3
Changed lines of the file:
@@
 $EndDescr
 $Comp
-L Logic_Programmable:GAL16V8 IC2
+L Logic_Programmable:GAL16V8 IC3
 U 1 1 5EAF7BFD
 P 7100 2050
-F 0 "IC2" H 7100 2931 50  0000 C CNN
+F 0 "IC3" H 7100 2931 50  0000 C CNN
 F 1 "ATF16V8BQL-15" H 7100 2840 50  0000 C CNN
 F 2 "Package_DIP:DIP-20_W7.62mm_LongPads" H 7100 2050 50  0001 C CNN
@@
 ASEL
 $Comp
-L Logic_Programmable:GAL16V8 IC1
+L Logic_Programmable:GAL16V8 IC2
 U 1 1 5EAF6AE7
 P 4800 2050
-F 0 "IC1" H 4800 2931 50  0000 C CNN
+F 0 "IC2" H 4800 2931 50  0000 C CNN
 F 1 "ATF16V8BQL-15" H 4800 2840 50  0000 C CNN
 F 2 "Package_DIP:DIP-20_W7.62mm_LongPads" H 4800 2050 50  0001 C CNN
@@
 	10100 1300 10100 1700
 $Comp
-L rosco_m68k:V9958 IC3
+L rosco_m68k:V9958 IC1
 U 1 1 5EDA9097
 P 9850 3200
-F 0 "IC3" H 9850 4881 50  0000 C CNN
+F 0 "IC1" H 9850 4881 50  0000 C CNN
 F 1 "V9958" H 9850 4790 50  0000 C CNN
 F 2 "rosco_m68k:sdip64" H 9850 3750 50  0001 C CNN

Commit message: Add jumper to support 1.2 mainboard
Parts:
- added JP1: Jumper, rosco_m68k:pin-1X02, symbol Device:Jumper
Connections:
- net VDTACK: now reaches IC2.14 (IO6)
- net VDTACK: now also JP1.1
- net DTACK: now reaches J1.58 (Pin_58)
- net DTACK: now also JP1.2
- no-connect marks 46 -> 44
Other:
- note removed: "Pin 14 can generate IODTACK"
Changed lines of the file:
@@
 NoConn ~ 2000 3500
 NoConn ~ 2000 3600
-NoConn ~ 2000 3700
 Text Notes 1250 4200 0    50   ~ 0
 Note - Inverted layout!
@@
 Text GLabel 8600 2350 1    50   UnSpc ~ 0
 VCC
-NoConn ~ 5300 2050
-Text Notes 5600 2650 1    50   ~ 0
-Pin 14 can generate IODTACK
 Text GLabel 4750 5200 0    50   Input ~ 0
 VA5
@@
 Wire Wire Line
 	6400 4150 6400 3950
+Text GLabel 5300 2050 2    50   3State ~ 0
+VDTACK
+Text GLabel 2000 3700 2    50   3State ~ 0
+DTACK
+$Comp
+L Device:Jumper JP1
+U 1 1 5F36AC4F
+P 7150 5750
+F 0 "JP1" H 7150 6014 50  0000 C CNN
+F 1 "Jumper" H 7150 5923 50  0000 C CNN
+F 2 "rosco_m68k:pin-1X02" H 7150 5750 50  0001 C CNN
+F 3 "~" H 7150 5750 50  0001 C CNN
+	1    7150 5750
+	1    0    0    -1
+$EndComp
+Wire Wire Line
+	6850 5750 6550 5750
+Wire Wire Line
+	7450 5750 7750 5750
+Text GLabel 6550 5750 0    50   3State ~ 0
+VDTACK
+Text GLabel 7750 5750 2    50   3State ~ 0
+DTACK
 $EndSCHEMATC
