File: bus-board/design/kicad/r0/roscbus01/roscbus01.sch (KiCad schematic (older format))
At the start: 38 parts, among them J1 Conn_01x03_Male, J2 Screw_Terminal_01x02, J3 Jack-DC, J4 USB_B_Micro, SW1 POWER, U1 L7805

Commit message: Add BOM
Parts:
- R1: value 330R -> 1K
Changed lines of the file:
@@
 P 6200 6100
 F 0 "R1" V 5993 6100 50  0000 C CNN
-F 1 "330R" V 6084 6100 50  0000 C CNN
+F 1 "1K" V 6084 6100 50  0000 C CNN
 F 2 "rosco_m68k:R-0207_10" V 6130 6100 50  0001 C CNN
 F 3 "~" H 6200 6100 50  0001 C CNN
@@
 	1000 6950 1000 7350
 Wire Wire Line
-	1700 6650 1900 6650
-Wire Wire Line
 	1600 7400 2050 7400
 Wire Wire Line
@@
 	1    0    0    -1
 $EndComp
-Connection ~ 1900 6650
-Wire Wire Line
-	1900 6650 2250 6650
 Wire Wire Line
 	5000 7100 5650 7100
@@
 Wire Wire Line
 	4000 7100 4100 7100
+Wire Wire Line
+	1700 6650 2250 6650
 $EndSCHEMATC

Commit message: Fix #7
Parts:
- H1, H2, H3, H4, H5, H6, H7, H8: footprint MountingHole:MountingHole_2.7mm_M2.5 -> MountingHole:MountingHole_3.2mm_M3
Changed lines of the file:
@@
 F 0 "H1" H 3600 696 50  0000 L CNN
 F 1 "MountingHole" H 3600 605 50  0000 L CNN
-F 2 "MountingHole:MountingHole_2.7mm_M2.5" H 3500 650 50  0001 C CNN
+F 2 "MountingHole:MountingHole_3.2mm_M3" H 3500 650 50  0001 C CNN
 F 3 "~" H 3500 650 50  0001 C CNN
 	1    3500 650
@@
 F 0 "H2" H 4300 696 50  0000 L CNN
 F 1 "MountingHole" H 4300 605 50  0000 L CNN
-F 2 "MountingHole:MountingHole_2.7mm_M2.5" H 4200 650 50  0001 C CNN
+F 2 "MountingHole:MountingHole_3.2mm_M3" H 4200 650 50  0001 C CNN
 F 3 "~" H 4200 650 50  0001 C CNN
 	1    4200 650
@@
 F 0 "H3" H 5000 696 50  0000 L CNN
 F 1 "MountingHole" H 5000 605 50  0000 L CNN
-F 2 "MountingHole:MountingHole_2.7mm_M2.5" H 4900 650 50  0001 C CNN
+F 2 "MountingHole:MountingHole_3.2mm_M3" H 4900 650 50  0001 C CNN
 F 3 "~" H 4900 650 50  0001 C CNN
 	1    4900 650
@@
 F 0 "H4" H 5700 696 50  0000 L CNN
 F 1 "MountingHole" H 5700 605 50  0000 L CNN
-F 2 "MountingHole:MountingHole_2.7mm_M2.5" H 5600 650 50  0001 C CNN
+F 2 "MountingHole:MountingHole_3.2mm_M3" H 5600 650 50  0001 C CNN
 F 3 "~" H 5600 650 50  0001 C CNN
 	1    5600 650
@@
 F 0 "H5" H 6400 696 50  0000 L CNN
 F 1 "MountingHole" H 6400 605 50  0000 L CNN
-F 2 "MountingHole:MountingHole_2.7mm_M2.5" H 6300 650 50  0001 C CNN
+F 2 "MountingHole:MountingHole_3.2mm_M3" H 6300 650 50  0001 C CNN
 F 3 "~" H 6300 650 50  0001 C CNN
 	1    6300 650
@@
 F 0 "H6" H 7100 696 50  0000 L CNN
 F 1 "MountingHole" H 7100 605 50  0000 L CNN
-F 2 "MountingHole:MountingHole_2.7mm_M2.5" H 7000 650 50  0001 C CNN
+F 2 "MountingHole:MountingHole_3.2mm_M3" H 7000 650 50  0001 C CNN
 F 3 "~" H 7000 650 50  0001 C CNN
 	1    7000 650
@@
 F 0 "H8" H 8600 696 50  0000 L CNN
 F 1 "MountingHole" H 8600 605 50  0000 L CNN
-F 2 "MountingHole:MountingHole_2.7mm_M2.5" H 8500 650 50  0001 C CNN
+F 2 "MountingHole:MountingHole_3.2mm_M3" H 8500 650 50  0001 C CNN
 F 3 "~" H 8500 650 50  0001 C CNN
 	1    8500 650
@@
 F 0 "H7" H 7850 696 50  0000 L CNN
 F 1 "MountingHole" H 7850 605 50  0000 L CNN
-F 2 "MountingHole:MountingHole_2.7mm_M2.5" H 7750 650 50  0001 C CNN
+F 2 "MountingHole:MountingHole_3.2mm_M3" H 7750 650 50  0001 C CNN
 F 3 "~" H 7750 650 50  0001 C CNN
 	1    7750 650

Commit message: Bus revision 3
Parts:
- removed D1: BAT43, Diode_THT:D_DO-35_SOD27_P7.62mm_Horizontal, symbol Diode:BAT43
Connections:
- net VCC: now also C8.1, JP4.2, JP5.2, U1.3 (OUT)
Changed lines of the file:
@@
 encoding utf-8
 Sheet 1 1
-Title ""
-Date ""
-Rev ""
-Comp ""
-Comment1 ""
-Comment2 ""
+Title "ROSCO_M68K LOCAL BUS BACKPLANE"
+Date "2020-08-13"
+Rev "2"
+Comp "The Really Old-School Company Limited"
+Comment1 "Open Source Hardware licenced under CERN Open Hardware Licence"
+Comment2 "Copyright 2020 Ross Bamford and Contributors"
 Comment3 ""
 Comment4 ""
@@
 Text Notes 1050 850  0    50   ~ 0
 Recommended\nComputer Connection
-$Comp
-L Diode:BAT43 D1
-U 1 1 5EBDCC17
-P 5800 7100
-F 0 "D1" H 5800 6884 50  0000 C CNN
-F 1 "BAT43" H 5800 6975 50  0000 C CNN
-F 2 "Diode_THT:D_DO-35_SOD27_P7.62mm_Horizontal" H 5800 6925 50  0001 C CNN
-F 3 "http://www.vishay.com/docs/85660/bat42.pdf" H 5800 7100 50  0001 C CNN
-	1    5800 7100
-	-1   0    0    1
-$EndComp
-Wire Wire Line
-	5950 7100 6250 7100
 Text Notes 4250 7500 0    50   ~ 0
 Optional
@@
 	1    0    0    -1
 $EndComp
-Wire Wire Line
-	5000 7100 5650 7100
 Connection ~ 4000 7100
 Wire Wire Line
@@
 Wire Wire Line
 	1700 6650 2250 6650
+Wire Wire Line
+	5000 7100 6250 7100
 $EndSCHEMATC
