File: mc68681-duart/mc68681-duart-basic/design/kicad/mc68681-basic/mc68681-basic.kicad_pcb (KiCad board)
At the start: 4 copper layers, 80 x 110 mm, 36 parts, among them IC1 XR68C681CJTR-F, IC2 74HCT245, IC3 74HCT245, IC4 74HCT245, IC5 74125, IC6 IC6_DECO.PLD, IC7 IC7_UART_.PLD, J1 Conn_02x32_Odd_Even, J2 EXTBUS, J3 UART_A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

Commit message: Add updated CAM outputs and PDF etc
Parts:
- removed the REF** at (59.0, 129.4)
- added REF** (x2): SM-rosco_m68k_logo, rosco_m68k:SM-rosco_m68k_logo, F.Cu at (56.0, 144.0)
